File: PCB/MacroPed_foot/MacroPed_foot.kicad_sch (KiCad schematic)
At the start: 6 parts, among them J9 Conn_01x02_Socket, SW1 SW_SPST

Commit message: Moved JST connector to edge of footboard
Signed-off-by: Devnol <pgkoutsoumanis@gmail.com>
Parts:
- H1, H2, H3, H4: now left out of the parts list
- J9: LCSC Part # (none) -> C173752
- SW1: LCSC Part # (none) -> C5156480
Changed lines of the file:
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@@
   )
   (symbol (lib_id "Mechanical:MountingHole") (at 57.785 34.925 0) (unit 1)
-    (in_bom yes) (on_board yes) (dnp no) (fields_autoplaced)
+    (in_bom no) (on_board yes) (dnp no) (fields_autoplaced)
     (property "Reference" "H2" (at 60.325 33.655 0)
       (effects (font (size 1.27 1.27)) (justify left))
@@
     )
     (property "Datasheet" "~" (at 57.785 34.925 0)
+      (effects (font (size 1.27 1.27)) hide)
+    )
+    (property "LCSC Part #" "" (at 57.785 34.925 0)
       (effects (font (size 1.27 1.27)) hide)
     )
@@
       (effects (font (size 1.27 1.27)) hide)
     )
+    (property "LCSC Part #" "C5156480" (at 49.53 48.26 0)
+      (effects (font (size 1.27 1.27)) hide)
+    )
     (pin "1")
     (pin "2")
@@
   )
   (symbol (lib_id "Mechanical:MountingHole") (at 57.785 59.69 0) (unit 1)
-    (in_bom yes) (on_board yes) (dnp no) (fields_autoplaced)
+    (in_bom no) (on_board yes) (dnp no) (fields_autoplaced)
     (property "Reference" "H3" (at 60.96 58.42 0)
       (effects (font (size 1.27 1.27)) (justify left))
@@
       (effects (font (size 1.27 1.27)) hide)
     )
+    (property "LCSC Part #" "" (at 57.785 59.69 0)
+      (effects (font (size 1.27 1.27)) hide)
+    )
     (instances
       (project "MacroPed_foot"
@@
   )
   (symbol (lib_id "Mechanical:MountingHole") (at 40.64 59.69 0) (unit 1)
-    (in_bom yes) (on_board yes) (dnp no) (fields_autoplaced)
+    (in_bom no) (on_board yes) (dnp no) (fields_autoplaced)
     (property "Reference" "H4" (at 43.18 59.69 0)
       (effects (font (size 1.27 1.27)) (justify left))
@@
       (effects (font (size 1.27 1.27)) hide)
     )
+    (property "LCSC Part #" "" (at 40.64 59.69 0)
+      (effects (font (size 1.27 1.27)) hide)
+    )
     (instances
       (project "MacroPed_foot"
@@
   )
   (symbol (lib_id "Mechanical:MountingHole") (at 40.64 34.925 0) (unit 1)
-    (in_bom yes) (on_board yes) (dnp no) (fields_autoplaced)
+    (in_bom no) (on_board yes) (dnp no) (fields_autoplaced)
     (property "Reference" "H1" (at 43.18 33.655 0)
       (effects (font (size 1.27 1.27)) (justify left))
@@
     )
     (property "Datasheet" "~" (at 40.64 34.925 0)
+      (effects (font (size 1.27 1.27)) hide)
+    )
+    (property "LCSC Part #" "" (at 40.64 34.925 0)
       (effects (font (size 1.27 1.27)) hide)
     )
@@
       (effects (font (size 1.27 1.27)) hide)
     )
+    (property "LCSC Part #" "C173752" (at 46.99 38.1 0)
+      (effects (font (size 1.27 1.27)) hide)
+    )
